File: RC1980 CPU/RC1980 CPU.kicad_pcb (KiCad board)
At the start: 2 copper layers, 1073 parts

Commit message: Front tracks
Parts:
- added REF**: PAD, PAD:PAD, F.Cu at (124.5, 142.2)
- added REF**: PAD, PAD:PAD, F.Cu at (106.7, 96.5)
- added REF**: PAD, PAD:PAD, F.Cu at (137.2, 119.4)
- added REF**: PAD, PAD:PAD, F.Cu at (137.2, 114.3)
- moved REF** 2.54 mm to (188.0, 94.0)
Routing:
- net (no net): track 5.08 -> 3886.4 mm
Other:
- net class Default: clearance 0.2 -> 0.1; trace_width 0.25 -> 0.1
- net class Power added: clearance 0.2, trace_width 0.25, via_dia 0.6, via_drill 0.4
- net class Signal added: clearance 0.1, trace_width 0.1, via_dia 0.6, via_drill 0.4
- rule trace_clearance: 0.2 -> 0.1
- rule trace_min: 0.2 -> 0.1

Commit message: Back tracks
Routing:
- net (no net): track 3886.4 -> 7359.5 mm

Commit message: Labels
Other:
- board text added: "+5"
- board text added: "+5V"
- board text added: "1"
- board text added: "2"
- board text added: "3"
- board text added: "4"
- board text added: "5"
- board text added: "6"
- board text added: "7"
- board text added: "8"
- board text added: "9"
- board text added: "BUS"
- board text added: "C4"
- board text added: "C5"
- board text added: "CR1"
- board text added: "CR2"
- board text added: "GND"
- board text added: "INPUT"
- board text added: "LOAD"
- board text added: "M10"
- board text added: "M11"
- board text added: "M12"
- board text added: "M13"
- board text added: "M14"
- board text added: "M15"
- board text added: "M20"
- board text added: "M3"
- board text added: "M4"
- board text added: "M5"
- board text added: "M6"
- board text added: "M7"
- board text added: "M8"
- board text added: "M9"
- board text added: "MP C"
- board text added: "MP NC"
- board text added: "Q"
- board text added: "R10"
- board text added: "R4"
- board text added: "R5"
- board text added: "R6"
- board text added: "R7"
- board text added: "R8"
- board text added: "R9"
- board text added: "RUN"
- board text added: "X1"
- board text added: "X2"
- board text added: "X3"
- board text added: "X4"
- board text added: "Y1"
- board text added: "Y2"
- board text added: "Y3"
- board text added: "Y4"

Commit message: Gerber export
Parts:
- added REF**: 1pin, mounting:1pin, F.Cu at (95.9, 49.5)
- added REF**: 1pin, mounting:1pin, F.Cu at (88.3, 49.5)
- added REF**: 1pin, mounting:1pin, F.Cu at (95.9, 140.3)
- added REF**: 1pin, mounting:1pin, F.Cu at (88.3, 140.3)
- added REF**: 1pin, mounting:1pin, F.Cu at (62.9, 49.5)
- added REF**: 1pin, mounting:1pin, F.Cu at (62.9, 140.3)
- added REF**: 1pin, mounting:1pin, F.Cu at (123.8, 49.5)
- added REF**: 1pin, mounting:1pin, F.Cu at (131.4, 49.5)
- added REF**: 1pin, mounting:1pin, F.Cu at (123.8, 140.3)
- added REF**: 1pin, mounting:1pin, F.Cu at (131.4, 140.3)
- added REF**: 1pin, mounting:1pin, F.Cu at (159.4, 140.3)
- added REF**: 1pin, mounting:1pin, F.Cu at (167.0, 140.3)
- added REF**: 1pin, mounting:1pin, F.Cu at (159.4, 49.5)
- added REF**: 1pin, mounting:1pin, F.Cu at (167.0, 49.5)
- added REF**: 1pin, mounting:1pin, F.Cu at (228.6, 49.5)
- added REF**: 1pin, mounting:1pin, F.Cu at (228.6, 140.3)
- moved REF** 27.6 mm to (64.1, 135.9)
- moved REF** 27.6 mm to (87.0, 135.9)
- moved REF** 27.6 mm to (81.9, 135.9)
- moved REF** 27.6 mm to (104.8, 135.9)
- moved REF** 27.6 mm to (109.9, 135.9)
- moved REF** 27.6 mm to (114.9, 135.9)
- moved REF** 27.6 mm to (140.3, 135.9)
- moved REF** 27.6 mm to (142.9, 135.9)
- moved REF** 27.6 mm to (148.0, 135.9)
- moved REF** 27.6 mm to (150.5, 135.9)
- moved REF** 27.6 mm to (61.6, 135.9)
- moved REF** 27.6 mm to (74.3, 135.9)
- moved REF** 27.6 mm to (69.2, 135.9)
- moved REF** 27.6 mm to (89.5, 135.9)
- moved REF** 27.6 mm to (66.7, 135.9)
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Other:
- board outline added: 173.4 x 98.4 mm
- board text added: "SECTION 1"
- board text added: "SECTION 2"
- board text added: "SECTION 3"
- board text added: "SECTION 4"
